Commit message: modify ojt_6

File: src/ojt_6/urdf/ojt-6.urdf (robot description, URDF)
Before this commit: robot ojt_6, 4 links, 3 joints
Links:
- removed link rear_laser
Joints:
- removed joint rear_laser_joint

Commit message: modify ojt_6

File: src/ojt_6/urdf/ojt-6.urdf (robot description, URDF)
Before this commit: robot ojt_6, 3 links, 2 joints
Links:
- removed link front_laser
- added link laser
Joints:
- removed joint front_laser_joint
- added joint laser_joint: type fixed, parent base_link, child laser, origin xyz=0.1455 0.067 0.03 rpy=0 0 0.7854

Commit message: test

File: src/ojt_6/urdf/ojt-6.urdf (robot description, URDF)
Before this commit: robot ojt_6, 3 links, 2 joints
Links:
- removed link laser
- added link laser_link
Joints:
- joint laser_joint: child laser -> laser_link

Commit message: modify ojt-6

File: src/ojt_6/urdf/ojt-6.urdf (robot description, URDF)
Before this commit: robot ojt_6, 3 links, 2 joints
Joints:
- joint laser_joint: origin xyz=0.1455 0.067 0.03 rpy=0 0 0.7854 -> xyz=-0.1455 -0.067 0.03 rpy=0 0 -2.3562
